File: PWMeter.kicad_pcb (KiCad board)
At the start: 2 copper layers, 100 x 50 mm, 20 parts, among them J1 TEST_1P, J2 TEST_1P, J3 TEST_1P, J4 TEST_1P, U1 LM317T, U2 MC78M05CDT, U4 Arduino_Nano

Commit message: minor changes on sylkmask
Parts:
- J5: renamed from  ; value (none) -> CONN_01X08
- P1, P5: renamed from  
- R3: value R -> 100R
- moved R3 2.50 mm to (112.2, 84.2)
Connections:
- R3 pad 1: Net-(J5-Pad4) -> Net-(J5-Pad3)
- U4 pad 29: Net-(R3-Pad2) -> Net-(J5-Pad4)
- U4 pad 30: Net-(J5-Pad3) -> Net-(R3-Pad2)
Routing:
- net Net-(J5-Pad4): track 2.48 -> 7.96 mm
- net Net-(J5-Pad3): track 7.96 -> 2.50 mm
Other:
- board text added: "RF POWER METER BY DL2SBA http://www.dl2sba.com/"
Changed lines of the file:
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@@
     (links 41)
     (no_connects 0)
-    (area 90.899999 68.825 191.100001 119.275)
+    (area 90.924999 68.924999 191.075001 119.075001)
     (thickness 1.6)
-    (drawings 14)
+    (drawings 15)
     (tracks 149)
     (zones 0)
@@
   )
   (setup
-    (last_trace_width 1.5)
+    (last_trace_width 1)
     (user_trace_width 0.5)
     (user_trace_width 1)
@@
       (net 11 "Net-(J5-Pad5)"))
     (pad 29 thru_hole oval (at -16.51 -7.62) (size 2 2.6) (drill 1.2) (layers *.Cu *.Mask F.SilkS)
+      (net 12 "Net-(J5-Pad4)"))
+    (pad 30 thru_hole oval (at -19.05 -7.62) (size 2 2.6) (drill 1.2) (layers *.Cu *.Mask F.SilkS)
       (net 16 "Net-(R3-Pad2)"))
-    (pad 30 thru_hole oval (at -19.05 -7.62) (size 2 2.6) (drill 1.2) (layers *.Cu *.Mask F.SilkS)
-      (net 13 "Net-(J5-Pad3)"))
     (model ../../../../../../Users/Marco/Documents/Kicad/Projets/dl2sba/arduino/arduino_nano.wrl
       (at (xyz -1 -0.4 -0.2))
@@
     (descr "Connector Headers with Friction Lock, 22-27-2021, http://www.molex.com/pdm_docs/sd/022272021_sd.pdf")
     (tags "connector molex kk_6410 22-27-2021")
-    (fp_text reference " " (at 1 -4.5 180) (layer F.SilkS)
-      (effects (font (size 1 1) (thickness 0.15)))
-    )
-    (fp_text value "16/9V  in" (at 1.27 4.5 180) (layer F.Fab)
+    (fp_text reference P1 (at 1 -4.5 180) (layer F.SilkS) hide
+      (effects (font (size 1 1) (thickness 0.15)))
+    )
+    (fp_text value "16/9V  in" (at 1.27 4.5 180) (layer F.Fab) hide
       (effects (font (size 1 1) (thickness 0.15)))
     )
@@
     (descr "Connector Headers with Friction Lock, 22-27-2041, http://www.molex.com/pdm_docs/sd/022272021_sd.pdf")
     (tags "connector molex kk_6410 22-27-2041")
-    (fp_text reference " " (at 4 4 180) (layer F.SilkS)
+    (fp_text reference P5 (at 4 4 180) (layer F.SilkS) hide
       (effects (font (size 1.5 1.5) (thickness 0.15)))
     )
@@
     (descr "Mounting Hole 3.2mm, M3")
     (tags "mounting hole 3.2mm m3")
-    (fp_text reference J1 (at 0 -4.2) (layer F.SilkS)
-      (effects (font (size 1 1) (thickness 0.15)))
-    )
-    (fp_text value TEST_1P (at 0 4.2) (layer F.Fab)
+    (fp_text reference J1 (at 0 -4.2) (layer F.SilkS) hide
+      (effects (font (size 1 1) (thickness 0.15)))
+    )
+    (fp_text value TEST_1P (at 0 4.2) (layer F.Fab) hide
       (effects (font (size 1 1) (thickness 0.15)))
     )
@@
     (descr "Mounting Hole 3.2mm, M3")
     (tags "mounting hole 3.2mm m3")
-    (fp_text reference J2 (at 0 -4.2) (layer F.SilkS)
-      (effects (font (size 1 1) (thickness 0.15)))
-    )
-    (fp_text value TEST_1P (at 0 4.2) (layer F.Fab)
+    (fp_text reference J2 (at 0 -4.2) (layer F.SilkS) hide
+      (effects (font (size 1 1) (thickness 0.15)))
+    )
+    (fp_text value TEST_1P (at 0 4.2) (layer F.Fab) hide
       (effects (font (size 1 1) (thickness 0.15)))
     )
@@
     (descr "Mounting Hole 3.2mm, M3")
     (tags "mounting hole 3.2mm m3")
-    (fp_text reference J3 (at 0 -4.2) (layer F.SilkS)
-      (effects (font (size 1 1) (thickness 0.15)))
-    )
-    (fp_text value TEST_1P (at 0 4.2) (layer F.Fab)
+    (fp_text reference J3 (at 0 -4.2) (layer F.SilkS) hide
+      (effects (font (size 1 1) (thickness 0.15)))
+    )
+    (fp_text value TEST_1P (at 0 4.2) (layer F.Fab) hide
       (effects (font (size 1 1) (thickness 0.15)))
     )
@@
     (at 116 80.5)
     (descr "8 pin vert. connector, Molex KK100 series")
-    (fp_text reference " " (at 8 -6.5) (layer F.SilkS)
+    (fp_text reference J5 (at 8 -6.5) (layer F.SilkS) hide
       (effects (font (thickness 0.3048)))
     )
-    (fp_text value " " (at 0 4.56946) (layer F.SilkS)
+    (fp_text value CONN_01X08 (at 0 4.56946) (layer F.SilkS) hide
       (effects (font (thickness 0.3048)))
     )
@@
   )
   (module Resistors_SMD:R_0805_HandSoldering (layer B.Cu)
-    (at 114.75 84.25 270)
+    (at 112.25 84.25 270)
     (descr "Resistor SMD 0805, hand soldering")
     (tags "resistor 0805")
@@
       (effects (font (size 1 1) (thickness 0.15)) (justify mirror))
     )
-    (fp_text value R (at 0 -1.75 270) (layer B.Fab)
+    (fp_text value 100R (at 0 -1.75 270) (layer B.Fab)
       (effects (font (size 1 1) (thickness 0.15)) (justify mirror))
     )
@@
     (fp_line (start 2.35 -0.9) (end -2.35 -0.9) (layer B.CrtYd) (width 0.05))
     (pad 1 smd rect (at -1.35 0 270) (size 1.5 1.3) (layers B.Cu B.Paste B.Mask)
-      (net 12 "Net-(J5-Pad4)"))
+      (net 13 "Net-(J5-Pad3)"))
     (pad 2 smd rect (at 1.35 0 270) (size 1.5 1.3) (layers B.Cu B.Paste B.Mask)
       (net 16 "Net-(R3-Pad2)"))
@@
       (rotate (xyz 0 0 0))
     )
+  )
+  (gr_text "RF POWER METER BY DL2SBA\nhttp://www.dl2sba.com/" (at 118 110) (layer F.SilkS)
+    (effects (font (size 1.5 1.5) (thickness 0.3)))
   )
   (gr_text "12Vcc\nGND" (at 170.5 78.5 90) (layer B.SilkS)
@@
   (segment (start 117.27 80.4238) (end 117.27 88.37) (width 1) (layer F.Cu) (net 11))
   (segment (start 117.27 88.37) (end 117.28 88.38) (width 0.5) (layer F.Cu) (net 11))
-  (segment (start 114.75 82.9) (end 114.75 80.4438) (width 0.5) (layer B.Cu) (net 12))
-  (segment (start 114.75 80.4438) (end 114.73 80.4238) (width 0.5) (layer B.Cu) (net 12))
-  (segment (start 112.19 80.4238) (end 112.19 88.37) (width 1) (layer F.Cu) (net 13))
-  (segment (start 112.19 88.37) (end 112.2 88.38) (width 0.5) (layer F.Cu) (net 13))
+  (segment (start 114.73 80.4238) (end 114.73 88.37) (width 1) (layer F.Cu) (net 12))
+  (segment (start 114.73 88.37) (end 114.74 88.38) (width 1) (layer F.Cu) (net 12))
+  (segment (start 112.19 80.4238) (end 112.19 82.84) (width 1) (layer B.Cu) (net 13))
+  (segment (start 112.19 82.84) (end 112.25 82.9) (width 1) (layer B.Cu) (net 13))
   (segment (start 122.36 103.62) (end 122.36 105.14) (width 1) (layer F.Cu) (net 14))
   (segment (start 121.5 76) (end 124.89 79.39) (width 1) (layer F.Cu) (net 14))
@@
   (segment (start 119.81 80.4238) (end 119.81 88.37) (width 1) (layer F.Cu) (net 15))
   (segment (start 119.81 88.37) (end 119.82 88.38) (width 0.5) (layer F.Cu) (net 15))
-  (segment (start 114.75 85.6) (end 114.75 88.37) (width 0.5) (layer B.Cu) (net 16))
-  (segment (start 114.75 88.37) (end 114.74 88.38) (width 0.5) (layer B.Cu) (net 16))
+  (segment (start 112.25 85.6) (end 112.25 88.33) (width 1) (layer B.Cu) (net 16))
+  (segment (start 112.19 88.37) (end 112.2 88.38) (width 0.5) (layer F.Cu) (net 16))
   (zone (net 2) (net_name GND) (layer B.Cu) (hatch edge 0.508)
     (connect_pads (clearance 0.508))
